File: KiCad PCBs/HIDman-micro/pcb.kicad_pcb (KiCad board)
At the start: 2 copper layers, 10.8 x 12.7 mm, 13 parts, among them J1 Conn_02x04_Odd_Even, P1 USB_A, SW1 SW_Push, U1 CH559T

Commit message: Tweak pad/track size/spacing
Parts:
- U1: footprint Package_SO:SSOP-20_5.3x7.2mm_P0.65mm -> USER_Footprints:SSOP-20_5.3x7.2mm_P0.65mm
Other:
- net class Default: clearance 0.15 -> 0.1778
- rule trace_clearance: 0.15 -> 0.1778
