File: KiCad PCBs/DB9-to-TTL/adapter.kicad_pcb (KiCad board)
At the start: 2 copper layers, 13.8 x 13.2 mm, 8 parts, among them J1 Conn_01x06, P1 DB9_Female, U1 MAX3232

Commit message: More verbose DB9-TTL Schematic
Parts:
- C2: value 1u -> 100n
Connections:
- net Net-(P1-Pad2) renamed /RXD_232
- net Net-(P1-Pad3) renamed /TXD_232
- net Net-(P1-Pad7) renamed /RTS_232
- net Net-(P1-Pad8) renamed /CTS_232
- P1 pad 1: Net-(P1-Pad1) -> (no net)
- P1 pad 4: Net-(P1-Pad4) -> (no net)
- P1 pad 6: Net-(P1-Pad6) -> (no net)
- P1 pad 9: Net-(P1-Pad9) -> (no net)
